Commit message: Updated urdf to seperate base link from frame

File: src/descriptors/urdf/open_dubs_description.urdf (robot description, URDF)
Before this commit: robot open_dubs, 2 links, 1 joints
Links:
- added link frame_link; collision box size=${frame_length} ${frame_width} ${frame_height}; visual box size=${frame_length} ${frame_width} ${frame_height}
- link base_link: geometry 
Joints:
- added joint frame_joint: type fixed, parent base_link, child frame_link, origin xyz=0.0 0.0 ${frame_height/2.0} rpy=0.0 0.0 0.0
- joint base_joint: origin xyz=0.0 0.0 ${-(wheel_radius+wheel_zoff)} rpy=0 0 0 -> xyz=0.0 0.0 ${frame_height/2.0+wheel_zoff-wheel_radius} rpy=0 0 0
